Commit message: moved c++ side to recieve robot_plan_t messages instead of a stream of lcmt_robot_state_messages

File: drake/examples/bhpn_drake_interface/object_conversion_utils/generated_drake_objects/sodaA.urdf (robot description, URDF)
Before this commit: robot tableIkea2, 1 links, 0 joints
Links:
- removed link tableIkea2
- added link sodaA, mass 6.0; collision mesh filename=sodaA.obj; visual mesh filename=sodaA.obj
