Commit message: pr2 with joints for base movement allmost fully works with bhpn

File: drake/examples/bhpn_drake_interface/object_conversion_utils/generated_drake_objects/lowTable.urdf (robot description, URDF)
Before this commit: robot tableIkea2, 1 links, 0 joints
Links:
- removed link tableIkea2
- added link lowTable, mass 6.0; collision mesh filename=lowTable.obj; visual mesh filename=lowTable.obj

File: drake/examples/bhpn_drake_interface/object_conversion_utils/generated_drake_objects/objAA.urdf (robot description, URDF)
Before this commit: robot tableIkea2, 1 links, 0 joints
Links:
- removed link tableIkea2
- added link objAA, mass 6.0; collision mesh filename=objAA.obj; visual mesh filename=objAA.obj

File: drake/examples/bhpn_drake_interface/object_conversion_utils/generated_drake_objects/solidTable.urdf (robot description, URDF)
Before this commit: robot tableIkea2, 1 links, 0 joints
Links:
- removed link tableIkea2
- added link solidTable, mass 6.0; collision mesh filename=solidTable.obj; visual mesh filename=solidTable.obj
