Commit message: gave somewhat okay controller

File: drake/examples/bhpn_drake_interface/object_conversion_utils/generated_drake_objects/objA.urdf (robot description, URDF)
Before this commit: robot objA, 1 links, 0 joints
Links:
- link objA: mass 0.5 -> 1.0

File: drake/examples/bhpn_drake_interface/object_conversion_utils/generated_drake_objects/tableIkea1.urdf (robot description, URDF)
Before this commit: robot tableIkea1, 1 links, 0 joints
Links:
- link tableIkea1: mass 0.5 -> 5.0

File: drake/examples/bhpn_drake_interface/object_conversion_utils/template.urdf (robot description, URDF)
Before this commit: robot object_name, 1 links, 0 joints
Links:
- link object_name: mass 0.5 -> M

Commit message: updated everything

File: drake/examples/bhpn_drake_interface/object_conversion_utils/generated_drake_objects/objA.urdf (robot description, URDF)
Before this commit: robot objA, 1 links, 0 joints
Links:
- link objA: mass 1.0 -> 2.0

File: drake/examples/bhpn_drake_interface/object_conversion_utils/generated_drake_objects/tableIkea1.urdf (robot description, URDF)
Before this commit: robot tableIkea1, 1 links, 0 joints
Links:
- link tableIkea1: mass 5.0 -> 6.0

Commit message: picking works with movable base drake pr2 (kind of)

File: drake/examples/bhpn_drake_interface/object_conversion_utils/generated_drake_objects/objA.urdf (robot description, URDF)
Before this commit: robot objA, 1 links, 0 joints
Links:
- link objA: mass 2.0 -> 1.0

Commit message: now it pr2 picks up ordinary shape ... sometimes

File: drake/examples/bhpn_drake_interface/object_conversion_utils/generated_drake_objects/objA.urdf (robot description, URDF)
Before this commit: robot objA, 1 links, 0 joints
Links:
- link objA: mass 1.0 -> 0.015

File: drake/examples/bhpn_drake_interface/object_conversion_utils/generated_drake_objects/sodaA.urdf (robot description, URDF)
Before this commit: robot sodaA, 1 links, 0 joints
Links:
- link sodaA: mass 6.0 -> 0.015
