Commit message: added movable valkyrie fingers to urdf. annoying but hopefully worthwile

File: drake/examples/valkyrie/urdf/urdf/valkyrie.urdf (robot description, URDF)
Before this commit: robot valkyrie, 87 links, 86 joints
Joints:
- joint leftIndexFingerPitch1: limit (none) -> lower=-0.08726646255 upper=0.08726646255 effort=10 velocity=1; type fixed -> revolute
- joint leftIndexFingerPitch2: limit (none) -> lower=-1.65806278845 upper=0.1745329251 effort=10 velocity=1; type fixed -> revolute
- joint leftIndexFingerPitch3: limit (none) -> lower=-1.9198621761 upper=0 effort=10 velocity=1; type fixed -> revolute
- joint leftMiddleFingerPitch1: limit (none) -> lower=-1.65806278845 upper=0.1745329251 effort=10 velocity=1; type fixed -> revolute
- joint leftMiddleFingerPitch2: limit (none) -> lower=-1.9198621761 upper=0 effort=10 velocity=1; type fixed -> revolute
- joint leftMiddleFingerPitch3: limit (none) -> lower=-1.5707963259 upper=0.1745329251 effort=10 velocity=1; type fixed -> revolute
- joint leftPinkyPitch1: limit (none) -> lower=-0.26179938765 upper=0 effort=10 velocity=1; type fixed -> revolute
- joint leftPinkyPitch2: limit (none) -> lower=-1.65806278845 upper=0.1745329251 effort=10 velocity=1; type fixed -> revolute
- joint leftPinkyPitch3: limit (none) -> lower=-1.9198621761 upper=0 effort=10 velocity=1; type fixed -> revolute
- joint leftThumbPitch1: axis 0 0 1 -> 1 0 0; limit (none) -> lower=-1.65806278845 upper=0.1745329251 effort=10 velocity=1; type fixed -> revolute
- joint leftThumbPitch2: axis 0 0 1 -> 1 0 0; limit (none) -> lower=-1.9198621761 upper=0 effort=10 velocity=1; type fixed -> revolute
- joint leftThumbPitch3: axis 0 0 1 -> 1 0 0; limit (none) -> lower=-1.5707963259 upper=0.1745329251 effort=10 velocity=1; type fixed -> revolute
- joint leftThumbRoll: axis 0 0 1 -> 0 1 0; limit (none) -> lower=-0.08726646255 upper=2.35619448885 effort=10 velocity=1; type fixed -> revolute
- joint rightIndexFingerPitch1: axis 0 0 1 -> 0 0 -1; limit (none) -> lower=-0.08726646255 upper=0.08726646255 effort=10 velocity=1; type fixed -> revolute
- joint rightIndexFingerPitch2: axis 0 0 1 -> 0 0 -1; limit (none) -> lower=-1.65806278845 upper=0.1745329251 effort=10 velocity=1; type fixed -> revolute
- joint rightIndexFingerPitch3: axis 0 0 1 -> 0 0 -1; limit (none) -> lower=-1.9198621761 upper=0 effort=10 velocity=1; type fixed -> revolute
- joint rightMiddleFingerPitch1: axis 0 0 1 -> 0 0 -1; limit (none) -> lower=-1.65806278845 upper=0.1745329251 effort=10 velocity=1; type fixed -> revolute
- joint rightMiddleFingerPitch2: axis 0 0 1 -> 0 0 -1; limit (none) -> lower=-1.9198621761 upper=0 effort=10 velocity=1; type fixed -> revolute
- joint rightMiddleFingerPitch3: axis 0 0 1 -> 0 0 -1; limit (none) -> lower=-1.5707963259 upper=0.1745329251 effort=10 velocity=1; type fixed -> revolute
- joint rightPinkyPitch1: axis 0 0 1 -> 0 0 -1; limit (none) -> lower=-0.26179938765 upper=0 effort=10 velocity=1; type fixed -> revolute
- joint rightPinkyPitch2: axis 0 0 1 -> 0 0 -1; limit (none) -> lower=-1.65806278845 upper=0.1745329251 effort=10 velocity=1; type fixed -> revolute
- joint rightPinkyPitch3: axis 0 0 1 -> 0 0 -1; limit (none) -> lower=-1.9198621761 upper=0 effort=10 velocity=1; type fixed -> revolute
- joint rightThumbPitch1: axis 0 0 1 -> -1 0 0; limit (none) -> lower=-1.65806278845 upper=0.1745329251 effort=10 velocity=1; type fixed -> revolute
- joint rightThumbPitch2: axis 0 0 1 -> -1 0 0; limit (none) -> lower=-1.9198621761 upper=0 effort=10 velocity=1; type fixed -> revolute
- joint rightThumbPitch3: axis 0 0 1 -> -1 0 0; limit (none) -> lower=-1.5707963259 upper=0.1745329251 effort=10 velocity=1; type fixed -> revolute
- joint rightThumbRoll: axis 0 0 1 -> 0 1 0; limit (none) -> lower=-0.08726646255 upper=2.35619448885 effort=10 velocity=1; type fixed -> revolute

File: drake/examples/valkyrie/urdf/urdf/valkyrie_A_sim_drake_one_neck_dof_wide_ankle_rom.urdf (robot description, URDF)
Before this commit: robot valkyrie, 87 links, 86 joints
Joints:
- joint leftPinkyPitch1: limit (none) -> lower=-0.26179938765 upper=0 effort=10 velocity=1
