Commit message: more changes with valkyrie to see if I can get visualization to work. Wasn't able to :(

File: drake/examples/valkyrie/urdf/urdf/valkyrie_A_sim_drake_one_neck_dof_wide_ankle_rom.urdf (robot description, URDF)
Before this commit: robot valkyrie, 87 links, 86 joints
Links:
- link hokuyo_link: geometry collision box size=0.08 0.06 0.04238; collision cylinder length=0.047 radius=0.024425
- link leftAnklePitchLink: geometry collision mesh filename=package://valkyrie/urdf/model/meshes/legs/lj5.vtp; visual mesh filename=package://valkyrie/urdf/model/meshes/legs/lj5.vtp
- link leftElbowPitchLink: geometry collision mesh filename=package://valkyrie/urdf/model/meshes/arms/aj4_left.vtp; visual mesh filename=package://valkyrie/urdf/model/meshes/arms/aj4_left.vtp
- link leftFoot: geometry collision box size=0.27 0.16 0.064; collision sphere radius=0.0
- link leftForearmLink: geometry collision mesh filename=package://valkyrie/urdf/model/meshes/arms/aj5_left.vtp; visual mesh filename=package://valkyrie/urdf/model/meshes/arms/aj5_left.vtp
- link leftHipPitchLink: geometry collision mesh filename=package://valkyrie/urdf/model/meshes/legs/lj3_left.vtp; visual mesh filename=package://valkyrie/urdf/model/meshes/legs/lj3_left.vtp
- link leftHipRollLink: geometry collision mesh filename=package://valkyrie/urdf/model/meshes/legs/lj2_left.vtp; visual mesh filename=package://valkyrie/urdf/model/meshes/legs/lj2_left.vtp
- link leftHipYawLink: geometry collision mesh filename=package://valkyrie/urdf/model/meshes/legs/lj1_left.vtp; visual mesh filename=package://valkyrie/urdf/model/meshes/legs/lj1_left.vtp
- link leftIndexFingerPitch1Link: geometry collision mesh filename=package://valkyrie/urdf/model/meshes/fingers/indexj1_left.v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; visual mesh filename=package://valkyrie/urdf/model/meshes/fingers/indexj1_left.v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
- link leftIndexFingerPitch2Link: geometry collision mesh filename=package://valkyrie/urdf/model/meshes/fingers/indexj2_left.v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; visual mesh filename=package://valkyrie/urdf/model/meshes/fingers/indexj2_left.v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
- link leftIndexFingerPitch3Link: geometry collision mesh filename=package://valkyrie/urdf/model/meshes/fingers/indexj3_left.v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; visual mesh filename=package://valkyrie/urdf/model/meshes/fingers/indexj3_left.v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
- link leftKneePitchLink: geometry collision mesh filename=package://valkyrie/urdf/model/meshes/legs/lj4_left.vtp; visual mesh filename=package://valkyrie/urdf/model/meshes/legs/lj4_left.vtp
- link leftMiddleFingerPitch1Link: geometry collision mesh filename=package://valkyrie/urdf/model/meshes/fingers/middlej1_left.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; visual mesh filename=package://valkyrie/urdf/model/meshes/fingers/middlej1_left.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
- link leftMiddleFingerPitch2Link: geometry collision mesh filename=package://valkyrie/urdf/model/meshes/fingers/middlej2_left.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; visual mesh filename=package://valkyrie/urdf/model/meshes/fingers/middlej2_left.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
- link leftMiddleFingerPitch3Link: geometry collision mesh filename=package://valkyrie/urdf/model/meshes/fingers/middlej3_left.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; visual mesh filename=package://valkyrie/urdf/model/meshes/fingers/middlej3_left.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
- link leftPalm: geometry collision mesh filename=package://valkyrie/urdf/model/meshes/arms/palm_left.vtp; visual mesh filename=package://valkyrie/urdf/model/meshes/arms/palm_left.vtp
- link leftPinkyPitch1Link: geometry collision mesh filename=package://valkyrie/urdf/model/meshes/fingers/pinkyj1_left.v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; visual mesh filename=package://valkyrie/urdf/model/meshes/fingers/pinkyj1_left.v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
- link leftPinkyPitch2Link: geometry collision mesh filename=package://valkyrie/urdf/model/meshes/fingers/pinkyj2_left.v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; visual mesh filename=package://valkyrie/urdf/model/meshes/fingers/pinkyj2_left.v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
- link leftPinkyPitch3Link: geometry collision mesh filename=package://valkyrie/urdf/model/meshes/fingers/pinkyj3_left.v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; visual mesh filename=package://valkyrie/urdf/model/meshes/fingers/pinkyj3_left.v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
- link leftShoulderPitchLink: geometry collision mesh filename=package://valkyrie/urdf/model/meshes/arms/aj1_left.vtp; visual mesh filename=package://valkyrie/urdf/model/meshes/arms/aj1_left.vtp
- link leftShoulderRollLink: geometry collision mesh filename=package://valkyrie/urdf/model/meshes/arms/aj2_left.vtp; visual mesh filename=package://valkyrie/urdf/model/meshes/arms/aj2_left.vtp
- link leftShoulderYawLink: geometry collision mesh filename=package://valkyrie/urdf/model/meshes/arms/aj3_left.vtp; visual mesh filename=package://valkyrie/urdf/model/meshes/arms/aj3_left.vtp
- link leftThumbPitch1Link: geometry collision mesh filename=package://valkyrie/urdf/model/meshes/fingers/thumbj2_left.v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; visual mesh filename=package://valkyrie/urdf/model/meshes/fingers/thumbj2_left.v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
- link leftThumbPitch2Link: geometry collision mesh filename=package://valkyrie/urdf/model/meshes/fingers/thumbj3_left.v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; visual mesh filename=package://valkyrie/urdf/model/meshes/fingers/thumbj3_left.v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
- link leftThumbPitch3Link: geometry collision mesh filename=package://valkyrie/urdf/model/meshes/fingers/thumbj4_left.v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; visual mesh filename=package://valkyrie/urdf/model/meshes/fingers/thumbj4_left.v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
- link leftThumbRollLink: geometry collision mesh filename=package://valkyrie/urdf/model/meshes/fingers/thumbj1_left.v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; visual mesh filename=package://valkyrie/urdf/model/meshes/fingers/thumbj1_left.v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
- link leftWristRollLink: geometry collision mesh filename=package://valkyrie/urdf/model/meshes/arms/aj6_left.vtp; visual mesh filename=package://valkyrie/urdf/model/meshes/arms/aj6_left.vtp
- link lowerNeckPitchLink: geometry collision mesh filename=package://valkyrie/urdf/model/meshes/head/neckj1.vtp; visual mesh filename=package://valkyrie/urdf/model/meshes/head/neckj1.vtp
- link neckYawLink: geometry collision mesh filename=package://valkyrie/urdf/model/meshes/head/neckj2.vtp; visual mesh filename=package://valkyrie/urdf/model/meshes/head/neckj2.vtp
- link pelvis: geometry collision mesh filename=package://valkyrie/urdf/model/meshes/pelvis/pelvis.vtp; visual mesh filename=package://valkyrie/urdf/model/meshes/pelvis/pelvis.vtp
- link rightAnklePitchLink: geometry collision mesh filename=package://valkyrie/urdf/model/meshes/legs/lj5.vtp; visual mesh filename=package://valkyrie/urdf/model/meshes/legs/lj5.vtp
- link rightElbowPitchLink: geometry collision mesh filename=package://valkyrie/urdf/model/meshes/arms/aj4_right.vtp; visual mesh filename=package://valkyrie/urdf/model/meshes/arms/aj4_right.vtp
- link rightFoot: geometry collision box size=0.27 0.16 0.064; collision sphere radius=0.0
- link rightForearmLink: geometry collision mesh filename=package://valkyrie/urdf/model/meshes/arms/aj5_right.vtp; visual mesh filename=package://valkyrie/urdf/model/meshes/arms/aj5_right.vtp
- link rightHipPitchLink: geometry collision mesh filename=package://valkyrie/urdf/model/meshes/legs/lj3_right.vtp; visual mesh filename=package://valkyrie/urdf/model/meshes/legs/lj3_right.vtp
- link rightHipRollLink: geometry collision mesh filename=package://valkyrie/urdf/model/meshes/legs/lj2_right.vtp; visual mesh filename=package://valkyrie/urdf/model/meshes/legs/lj2_right.vtp
- link rightHipYawLink: geometry collision mesh filename=package://valkyrie/urdf/model/meshes/legs/lj1_right.vtp; visual mesh filename=package://valkyrie/urdf/model/meshes/legs/lj1_right.vtp
- link rightIndexFingerPitch1Link: geometry collision mesh filename=package://valkyrie/urdf/model/meshes/fingers/indexj1_right.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; visual mesh filename=package://valkyrie/urdf/model/meshes/fingers/indexj1_right.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
- link rightIndexFingerPitch2Link: geometry collision mesh filename=package://valkyrie/urdf/model/meshes/fingers/indexj2_right.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; visual mesh filename=package://valkyrie/urdf/model/meshes/fingers/indexj2_right.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
- link rightIndexFingerPitch3Link: geometry collision mesh filename=package://valkyrie/urdf/model/meshes/fingers/indexj3_right.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; visual mesh filename=package://valkyrie/urdf/model/meshes/fingers/indexj3_right.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
- link rightKneePitchLink: geometry collision mesh filename=package://valkyrie/urdf/model/meshes/legs/lj4_right.vtp; visual mesh filename=package://valkyrie/urdf/model/meshes/legs/lj4_right.vtp
- link rightMiddleFingerPitch1Link: geometry collision mesh filename=package://valkyrie/urdf/model/meshes/fingers/middlej1_right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; visual mesh filename=package://valkyrie/urdf/model/meshes/fingers/middlej1_right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
- link rightMiddleFingerPitch2Link: geometry collision mesh filename=package://valkyrie/urdf/model/meshes/fingers/middlej2_right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; visual mesh filename=package://valkyrie/urdf/model/meshes/fingers/middlej2_right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
- link rightMiddleFingerPitch3Link: geometry collision mesh filename=package://valkyrie/urdf/model/meshes/fingers/middlej3_right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; visual mesh filename=package://valkyrie/urdf/model/meshes/fingers/middlej3_right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
- link rightPalm: geometry collision mesh filename=package://valkyrie/urdf/model/meshes/arms/palm_right.vtp; visual mesh filename=package://valkyrie/urdf/model/meshes/arms/palm_right.vtp
- link rightPinkyPitch1Link: geometry collision mesh filename=package://valkyrie/urdf/model/meshes/fingers/pinkyj1_right.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; visual mesh filename=package://valkyrie/urdf/model/meshes/fingers/pinkyj1_right.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
- link rightPinkyPitch2Link: geometry collision mesh filename=package://valkyrie/urdf/model/meshes/fingers/pinkyj2_right.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; visual mesh filename=package://valkyrie/urdf/model/meshes/fingers/pinkyj2_right.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
- link rightPinkyPitch3Link: geometry collision mesh filename=package://valkyrie/urdf/model/meshes/fingers/pinkyj3_right.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; visual mesh filename=package://valkyrie/urdf/model/meshes/fingers/pinkyj3_right.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
- link rightShoulderPitchLink: geometry collision mesh filename=package://valkyrie/urdf/model/meshes/arms/aj1_right.vtp; visual mesh filename=package://valkyrie/urdf/model/meshes/arms/aj1_right.vtp
- link rightShoulderRollLink: geometry collision mesh filename=package://valkyrie/urdf/model/meshes/arms/aj2_right.vtp; visual mesh filename=package://valkyrie/urdf/model/meshes/arms/aj2_right.vtp
- link rightShoulderYawLink: geometry collision mesh filename=package://valkyrie/urdf/model/meshes/arms/aj3_right.vtp; visual mesh filename=package://valkyrie/urdf/model/meshes/arms/aj3_right.vtp
- link rightThumbPitch1Link: geometry collision mesh filename=package://valkyrie/urdf/model/meshes/fingers/thumbj2_right.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; visual mesh filename=package://valkyrie/urdf/model/meshes/fingers/thumbj2_right.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
- link rightThumbPitch2Link: geometry collision mesh filename=package://valkyrie/urdf/model/meshes/fingers/thumbj3_right.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; visual mesh filename=package://valkyrie/urdf/model/meshes/fingers/thumbj3_right.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
- link rightThumbPitch3Link: geometry collision mesh filename=package://valkyrie/urdf/model/meshes/fingers/thumbj4_right.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; visual mesh filename=package://valkyrie/urdf/model/meshes/fingers/thumbj4_right.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
- link rightThumbRollLink: geometry collision mesh filename=package://valkyrie/urdf/model/meshes/fingers/thumbj1_right.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; visual mesh filename=package://valkyrie/urdf/model/meshes/fingers/thumbj1_right.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
- link rightWristRollLink: geometry collision mesh filename=package://valkyrie/urdf/model/meshes/arms/aj6_right.vtp; visual mesh filename=package://valkyrie/urdf/model/meshes/arms/aj6_right.vtp
- link torso: geometry collision mesh filename=package://valkyrie/urdf/model/meshes/torso/torso.vtp; visual mesh filename=package://valkyrie/urdf/model/meshes/torso/torso.vtp
- link torsoPitchLink: geometry collision mesh filename=package://valkyrie/urdf/model/meshes/torso/torsopitch.vtp; visual mesh filename=package://valkyrie/urdf/model/meshes/torso/torsopitch.vtp
- link torsoYawLink: geometry collision mesh filename=package://valkyrie/urdf/model/meshes/torso/torsoyaw.vtp; visual mesh filename=package://valkyrie/urdf/model/meshes/torso/torsoyaw.vtp
- link upperNeckPitchLink: geometry collision mesh filename=package://valkyrie/urdf/model/meshes/head/head_multisense_n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; visual mesh filename=package://valkyrie/urdf/model/meshes/head/head_multisense_n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
