Commit message: More work on val gripping.

File: drake/examples/Valkyrie/urdf/urdf/valkyrie_limited_finger_movement_no_collisions.urdf (robot description, URDF)
Before this commit: robot valkyrie, 87 links, 86 joints
Joints:
- joint leftThumbRoll: origin xyz=0.0049 0.0351 0.0228 rpy=-0.3491 2.3 0.0 -> xyz=0.0049 0.0351 0.0228 rpy=-0.3491 2.0 0.0
- joint rightThumbRoll: origin xyz=0.0049 -0.0351 0.0228 rpy=0.3491 2.3 0.0 -> xyz=0.0049 -0.0351 0.0228 rpy=0.3491 2.0 0.0
